File: 3-in-1dual.kicad_pcb (KiCad board)
At the start: 2 copper layers, 125 x 100 mm, 32 parts

Commit message: Update to KiCAD 9
Connections:
- net /~CF_CS renamed /~{CF_CS}
- net /~MEM_CS renamed /~{MEM_CS}
- net ~COM1_CS-0x3F8 renamed ~{COM1_CS-0x3F8}
- net ~COM2_CS-0x2F8 renamed ~{COM2_CS-0x2F8}
- net ~IOR renamed ~{IOR}
- net ~IOW renamed ~{IOW}
- net ~LPT2_CS-0x278 renamed ~{LPT2_CS-0x278}
- net ~MEMR renamed ~{MEMR}
- net ~MEMW renamed ~{MEMW}
- net ~RESET renamed ~{RESET}
Other:
- net class Default removed
