File: Multi-IO-Daughtercard.kicad_pcb (KiCad board)
At the start: 2 copper layers, 92 x 60 mm, 15 parts

Commit message: Update to KiCAD 9
Connections:
- net ~COM1_CS-0x3F8 renamed ~{COM1_CS-0x3F8}
- net ~COM2_CS-0x2F8 renamed ~{COM2_CS-0x2F8}
- net ~IOR renamed ~{IOR}
- net ~IOW renamed ~{IOW}
- net ~LPT2_CS-0x278 renamed ~{LPT2_CS-0x278}
- net ~RESET renamed ~{RESET}
Other:
- net class Default removed
